File: quad-v3/qv3_kicad/qv3_kicad.kicad_sch (KiCad schematic)
At the start: 0 parts

Commit message: steven schematic
Parts:
- added BZ1: Buzzer, symbol Device:Buzzer
- added R1, R2, R3: 1k, symbol Device:R
- added R4, R5, R6: 2k, symbol Device:R
- added U1: (no value), repo:esp32_30pin, symbol repo:ESP32_30Pin
- added U2: Adafruit 815 (PCA9685), repo:adafruit_pca9685, symbol repo:815
- added U3, U4: MAX7219, symbol Driver_LED:MAX7219
- added U5: HC-SR04 (RIGHT), repo:hc-sr04, symbol repo:HC-SR04
- added U6: HC-SR04 (MIDDLE), repo:hc-sr04, symbol repo:HC-SR04
- added U7: HC-SR04 (LEFT), repo:hc-sr04, symbol repo:HC-SR04
Connections:
- new net: R3.2, R6.1, U1.5 (GPIO14)
- new net: U3.24 (DOUT), U4.1 (DIN)
- new net: U1.23 (GPIO5), U3.12 (LOAD), U4.12 (LOAD)
- new net: U1.24 (GPIO18), U3.13 (CLK), U4.13 (CLK)
- new net: U1.16 (3.3v), U3.19 (V+), U4.19 (V+), U5.1 (VCC), U6.1 (VCC), U7.1 (VCC)
- new net: BZ1.1 (+), U1.8 (GPIO25)
- new net: U1.4 (GPIO12), U5.2 (TRIG), U6.2 (TRIG), U7.2 (TRIG)
- new net: R1.1, U5.3 (ECHO)
- new net: R2.1, U6.3 (ECHO)
- new net: R2.2, R5.1, U1.6 (GPIO27)
- new net: U1.26 (GPIO21), U2.SDA_1 (SDA), U2.SDA_2 (SDA)
- new net: U1.29 (GPIO22), U2.SCL_1 (SCL), U2.SCL_2 (SCL)
- new net: U1.30 (GPIO23), U3.1 (DIN)
- new net: R1.2, R4.1, U1.7 (GPIO26)
- new net: U2.OE_1 (~{OE}), U2.OE_2 (~{OE})
- new net: R3.1, U7.3 (ECHO)
- new net +5V: U1.1 (VIN)
- new net GND: BZ1.2 (-), R4.2, R5.2, R6.2, U1.17 (GND), U1.2 (GND), U2.GND_1 (GND), U2.GND_10 (GND), U2.GND_11 (GND), U2.GND_12 (GND), U2.GND_13 (GND), U2.GND_14 (GND), U2.GND_15 (GND), U2.GND_16 (GND), U2.GND_17 (GND), U2.GND_18 (GND), U2.GND_2 (GND), U2.GND_3 (GND), U2.GND_4 (GND), U2.GND_5 (GND), U2.GND_6 (GND), U2.GND_7 (GND), U2.GND_8 (GND), U2.GND_9 (GND), U3.4 (GND), U3.9 (GND), U4.4 (GND), U4.9 (GND), U5.4 (GND), U6.4 (GND), U7.4 (GND)
- new net V+: U2.V+_1 (V+), U2.V+_10 (V+), U2.V+_11 (V+), U2.V+_12 (V+), U2.V+_13 (V+), U2.V+_14 (V+), U2.V+_15 (V+), U2.V+_16 (V+), U2.V+_17 (V+), U2.V+_18 (V+), U2.V+_2 (V+), U2.V+_3 (V+), U2.V+_4 (V+), U2.V+_5 (V+), U2.V+_6 (V+), U2.V+_7 (V+), U2.V+_8 (V+), U2.V+_9 (V+)
- new net VCC: U2.VCC_1 (VCC), U2.VCC_2 (VCC)
